File: hardware/GloveMouse.brd (EAGLE design)
At the start: 44.4 x 46.5 mm, 44 parts, among them IC3 MCP73811/2, J1 USB MICRO, U1 ATMEGA32U4-XUAU, U4 MCP1825S-3302E/DB

Commit message: GloveMouse v2.3 all-in-one commit
Parts:
- removed GYRO: (no value), pinhead:1X05
- removed ON: GREEN, led:CHIP-LED0805
- removed R7: 10K, SmartPrj:R0603-ROUND
- removed SJ1: (no value), jumper:SJ
- removed STATUSLED: BLUE, led:CHIP-LED0805
- removed U$1: RN42, Tudor's_spankin'_library:RN42
- added C10, C17, C18: 0.1uF, resistor:C0603K
- added C12: 10uF, rcl:SMC_B
- added C14: 470nF, resistor:C0603K
- added C16: 10nF, resistor:C0603K
- added POWER: (no value), led:CHIP-LED0805
- added R10: 10K, resistor:R0603
- added R11, R12: 33K, resistor:R0603
- added STATUS: BLUE, led:CHIP-LED0805
- added U2: LPY403AL, Tudor's_spankin'_library:LGA28R50P8X6_500X400X100
- added U3: HC_05, SerialPortBluetooth:BLUETOOTH_SMD
- C1, C11, C15, C2, C3, C4, C5, C6, C7, C9: device SmartPrj:C0603-ROUND -> SmartPrj:C0603K
- C13: device rcl:C0603 -> rcl:C0603K
- R13, R8, R9: device SmartPrj:R0603-ROUND -> resistor:R0603
- moved C13 37.0 mm to (15.9, 43.5), turned to 270 degrees
- moved R21 34.7 mm to (41.7, 24.6)
- moved LED4 34.4 mm to (41.7, 28.7), turned to 180 degrees
- moved R23 33.4 mm to (39.7, 24.6), turned to 270 degrees
- moved R1 29.7 mm to (24.1, 10.5), turned to 270 degrees
- moved LED5 28.9 mm to (39.7, 28.7), turned to 180 degrees
- moved R2 28.5 mm to (33.4, 19.7), turned to 0 degrees
- moved C2 27.9 mm to (9.92, 12.2), turned to 270 degrees
- moved C15 10.8 mm to (9.98, 8.13), turned to 270 degrees
- moved R9 9.83 mm to (14.7, 8.13)
- moved R8 9.81 mm to (12.3, 8.14)
- moved R13 9.37 mm to (35.1, 10.1), turned to 90 degrees
- moved RESET_SW 7.53 mm to (40.1, 6.58)
- moved JP1 7.45 mm to (29.4, 11.6)
- moved R6 6.38 mm to (13.5, 40.2), turned to 270 degrees
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Connections:
- removed net ADC6: GYRO.3, U1.37
- removed net ADC7: GYRO.4, U1.36
- removed net HWB: R7.2, SJ1.1, U1.33
- removed net PF0: LED4.A, U1.41
- removed net PF1: LED5.A, U1.40
- new net 3.3V: U2.19, U2.9
- new net F1: C14.1, C16.1, U2.18
- new net F2: C16.2, R10.1, U2.17
- new net N$10: C18.2, R11.1, U2.16
- new net N$4: C14.2, R10.2
- new net N$6: R12.1, U2.1
- new net N$9: R11.2, U2.20
- new net PD0: LED5.A, U1.18
- new net PD1: LED4.A, U1.19
- new net X: U1.36, U2.14
- new net XOUT-1X2: C17.2, R12.2, U2.5
- new net Z: U1.37, U2.7
- net +3V3: now also C10.1, C12.+, U3.12; no longer GYRO.1, R7.1, U$1.11
- net AVCC: now also C5.2; no longer C5.1
- net GND: now also C10.2, C12.-, C17.1, C18.1, C5.1, POWER.C, U1.33, U2.24, U2.26, U2.27, U2.28, U3.13, U3.21, U3.22; no longer C5.2, GYRO.2, ON.C, SJ1.2, U$1.1, U$1.12, U$1.28, U$1.29
- net N$3: now also POWER.A; no longer ON.A
- net N$7: now also STATUS.A, U3.24; no longer STATUSLED.A, U$1.19
- net N$8: now also STATUS.C; no longer STATUSLED.C
- net RXD: now also U3.1; no longer U$1.14
- net TXD: now also U3.2; no longer U$1.13
Routing:
- net GND: track 346.6 -> 310.3 mm, vias 0 -> 1
- net +3V3: track 186.9 -> 216.7 mm, vias 2 -> 1
- net RXD: track 13.2 -> 35.2 mm
- net PD1: track 0.00 -> 18.9 mm
- net N$9: track 0.00 -> 18.1 mm
- net PD0: track 0.00 -> 16.1 mm
- net N$5: track 61.4 -> 46.5 mm
- net ADC7: track 13.6 -> 0.00 mm
- net ADC6: track 13.4 -> 0.00 mm
- net TXD: track 23.6 -> 33.2 mm
- net F2: track 0.00 -> 9.04 mm
- net RESET: track 37.7 -> 46.7 mm
- net RD-: track 10.0 -> 17.2 mm
- net D-: track 10.6 -> 3.42 mm
- net RD+: track 9.08 -> 16.2 mm
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Other:
- board text added: "X"
- board text added: "Y"

Commit message: GloveMouse v2.4 all-in-one commit
Parts:
- removed STATUS: BLUE, led:CHIP-LED0805
- removed U3: HC_05, SerialPortBluetooth:BLUETOOTH_SMD
- added STATUSLED: BLUE, led:CHIP-LED0805
- added U$1: RN42, Tudor's_spankin'_library:RN42
- LIPO: device pinhead:1X03 -> pinhead:1X02
- R2, R21, R23: value 1k -> 220
- moved LIPO 1.61 mm to (19.6, 42.5)
- moved R1 0.17 mm to (24.0, 10.4)
Connections:
- net +3V3: now also U$1.11; no longer U3.12
- net GND: now also U$1.1, U$1.12, U$1.28, U$1.29; no longer U3.13, U3.21, U3.22
- net N$7: now also STATUSLED.A, U$1.19; no longer STATUS.A, U3.24
- net N$8: now also STATUSLED.C; no longer STATUS.C
- net RXD: now also U$1.14; no longer U3.1
- net TXD: now also U$1.13; no longer U3.2
Routing:
- net GND: track 310.3 -> 337.8 mm, vias 1 -> 0
- net N$7: track 14.2 -> 24.9 mm
- net RESET: track 46.7 -> 42.6 mm
- net RXD: track 35.2 -> 38.3 mm
- net +3V3: track 216.7 -> 219.0 mm
- net N$5: track 46.5 -> 45.2 mm
