File: hardware/GloveMouse.sch (EAGLE design)
At the start: 44 parts, among them IC3 MCP73811/2, J1 USB MICRO, U1 ATMEGA32U4-XUAU, U4 MCP1825S-3302E/DB

Commit message: GloveMouse v2.3 all-in-one commit
Parts:
- removed GYRO: (no value), pinhead:PINHD-1X5
- removed ON: GREEN, led:LEDCHIP-LED0805
- removed R7: 10K, SmartPrj:R-EU_R0603
- removed SJ1: (no value), jumper:SJ
- removed STATUSLED: BLUE, led:LEDCHIP-LED0805
- removed U$1: RN42, Tudor's_spankin'_library:RN42
- added C10, C17, C18: 0.1uF, resistor:C-EUC0603K
- added C12: 10uF, rcl:CPOL-EUSMCB
- added C14: 470nF, resistor:C-EUC0603K
- added C16: 10nF, resistor:C-EUC0603K
- added POWER: (no value), led:LEDCHIP-LED0805
- added R10: 10K, resistor:R-EU_R0603
- added R11, R12: 33K, resistor:R-EU_R0603
- added STATUS: BLUE, led:LEDCHIP-LED0805
- added U2: LPY403AL, Tudor's_spankin'_library:LPY403AL
- added U3: HC_05, SerialPortBluetooth:HC_05
- C1, C11, C15, C2, C3, C4, C5, C6, C7, C9: device SmartPrj:C-EUC0603 -> SmartPrj:C-EUC0603K
- C13: device rcl:C-EUC0603 -> rcl:C-EUC0603K
- R13, R8, R9: device SmartPrj:R-EU_R0603 -> resistor:R-EU_R0603
Connections:
- removed net ADC6: GYRO.3, U1.(ADC6/TDO)PF6
- removed net ADC7: GYRO.4, U1.(ADC7/TDI)PF7
- removed net HWB: R7.2, SJ1.1, U1.(#HWB)PE2
- removed net PF0: LED4.A, U1.(ADC0)PF0
- removed net PF1: LED5.A, U1.(ADC1)PF1
- new net 3.3V: U2.VDD, U2.VDD_2
- new net F1: C14.1, C16.1, U2.FILTVDD
- new net F2: C16.2, R10.1, U2.VCONT
- new net N$10: C18.2, R11.1, U2.4XIN_X
- new net N$4: C14.2, R10.2
- new net N$6: R12.1, U2.OUT_Z
- new net N$9: R11.2, U2.OUT_X
- new net PD0: LED5.A, U1.(OC0B/SCL/INT0)PD0
- new net PD1: LED4.A, U1.(SDA/INT1)PD1
- new net X: U1.(ADC7/TDI)PF7, U2.4XOUT_X
- new net XOUT-1X2: C17.2, R12.2, U2.4XIN_Z
- new net Z: U1.(ADC6/TDO)PF6, U2.4XOUT_Z
- net +3V3: now also C10.1, C12.+, U3.3V3; no longer GYRO.1, R7.1, U$1.VDD
- net AVCC: now also C5.2; no longer C5.1
- net GND: now also C10.2, C12.-, C17.1, C18.1, C5.1, POWER.C, U1.(#HWB)PE2, U2.GND, U2.HP, U2.SLEEP/PD, U2.ST, U3.GND, U3.GND1, U3.GND2; no longer C5.2, GYRO.2, ON.C, SJ1.2, U$1.GND
- net N$3: now also POWER.A; no longer ON.A
- net N$7: now also STATUS.A, U3.PIO1; no longer STATUSLED.A, U$1.GPIO2
- net N$8: now also STATUS.C; no longer STATUSLED.C
- net RXD: now also U3.TX; no longer U$1.UART_TX
- net TXD: now also U3.RX; no longer U$1.UART_RX
Other:
- note added: "Gyroscope"
- note added: "ISP"
- note added: "Mouse buttons"
- note added: "Sensitivity"
- note added: "To Battery"
- note removed: "Gyro connector"
- note removed: "Sensitivity LEDs"
- note removed: "Sensitivity select button"
- note removed: "To Own Battery"
- note removed: "Touch buttons"
- note removed: "programator"
- moved on the sheet: C1, C11, C13, C15, C2, C3, C4, C5, C6, C7, C8, C9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

Commit message: GloveMouse v2.4 all-in-one commit
Parts:
- removed STATUS: BLUE, led:LEDCHIP-LED0805
- removed U3: HC_05, SerialPortBluetooth:HC_05
- added STATUSLED: BLUE, led:LEDCHIP-LED0805
- added U$1: RN42, Tudor's_spankin'_library:RN42
- LIPO: device pinhead:PINHD-1X3 -> pinhead:PINHD-1X2
- R2, R21, R23: value 1k -> 220
Connections:
- net +3V3: now also U$1.VDD; no longer U3.3V3
- net GND: now also U$1.GND; no longer U3.GND, U3.GND1, U3.GND2
- net N$7: now also STATUSLED.A, U$1.GPIO2; no longer STATUS.A, U3.PIO1
- net N$8: now also STATUSLED.C; no longer STATUS.C
- net RXD: now also U$1.UART_TX; no longer U3.TX
- net TXD: now also U$1.UART_RX; no longer U3.RX
Other:
- moved on the sheet: R1
