File: hardware/GloveMouse.sch (EAGLE design)
At the start: 46 parts, among them IC3 MCP73811/2, J1 USB MICRO, U1 ATMEGA32U4-XUAU, U4 MCP1825S-3302E/DB

Commit message: GloveMouse v2.1 all-in-one commit
Parts:
- removed PARANI: (no value), pinhead:PINHD-2X6
- added R1: 220, resistor:R-EU_R0603
- added STATUSLED: BLUE, led:LEDCHIP-LED0805
- added U$1: RN42, Tudor's_spankin'_library:RN42
Connections:
- new net N$7: STATUSLED.A, U$1.GPIO2
- new net N$8: R1.2, STATUSLED.C
- net +3V3: now also U$1.VDD; no longer PARANI.11
- net ADC10: now also LEFT_CLICK.2, R3.1; no longer R5.1, STAND-BY.2
- net ADC8: now also R5.1, STAND-BY.2; no longer LEFT_CLICK.2, R3.1
- net GND: now also R1.1, U$1.GND; no longer PARANI.1, PARANI.12, PARANI.9
- net RXD: now also U$1.UART_TX; no longer PARANI.3
- net TXD: now also U$1.UART_RX; no longer PARANI.5
Other:
- note removed: "Bluetooth connector"
Changed lines of the file:
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@@
 <part name="P+19" library="supply1" deviceset="+3V3" device="" value="+3V3"/>
 <part name="P+15" library="supply1" deviceset="+3V3" device="" value="+3V3"/>
-<part name="PARANI" library="pinhead" deviceset="PINHD-2X6" device=""/>
 <part name="GYRO" library="pinhead" deviceset="PINHD-1X7" device=""/>
+<part name="GND13" library="supply1" deviceset="GND" device=""/>
+<part name="P+1" library="supply1" deviceset="+3V3" device="" value="+3V3"/>
+<part name="U$1" library="Tudor's_spankin'_library" deviceset="RN42" device=""/>
+<part name="STATUSLED" library="led" deviceset="LED" device="CHIP-LED0805" value="BLUE"/>
+<part name="GND19" library="supply1" deviceset="GND" device=""/>
+<part name="R1" library="resistor" deviceset="R-EU_" device="R0603" value="220"/>
 </parts>
 <sheets>
@@
 <text x="175.26" y="74.93" size="1.778" layer="97">Sensitivity LEDs</text>
 <text x="223.52" y="99.06" size="1.778" layer="97">Gyro connector</text>
-<text x="223.52" y="66.04" size="1.778" layer="97">Bluetooth connector</text>
-<wire x1="220.98" y1="68.58" x2="220.98" y2="40.64" width="0.1524" layer="97" style="shortdash"/>
-<wire x1="220.98" y1="40.64" x2="266.7" y2="40.64" width="0.1524" layer="97" style="shortdash"/>
-<wire x1="266.7" y1="40.64" x2="266.7" y2="68.58" width="0.1524" layer="97" style="shortdash"/>
-<wire x1="266.7" y1="68.58" x2="220.98" y2="68.58" width="0.1524" layer="97" style="shortdash"/>
 </plain>
 <instances>
@@
 <attribute name="VALUE" x="212.725" y="104.14" size="1.778" layer="96" rot="R180"/>
 </instance>
-<instance part="PARANI" gate="A" x="243.84" y="53.34"/>
 <instance part="GYRO" gate="A" x="243.84" y="83.82"/>
+<instance part="GND13" gate="1" x="220.98" y="17.78"/>
+<instance part="P+1" gate="G$1" x="220.98" y="30.48" smashed="yes">
+<attribute name="VALUE" x="222.885" y="33.02" size="1.778" layer="96" rot="R180"/>
+</instance>
+<instance part="U$1" gate="G$1" x="195.58" y="2.54"/>
+<instance part="STATUSLED" gate="G$1" x="165.1" y="25.4" smashed="yes" rot="R270">
+<attribute name="NAME" x="157.988" y="29.464" size="1.778" layer="95"/>
+<attribute name="VALUE" x="163.068" y="22.225" size="1.778" layer="96"/>
+</instance>
+<instance part="GND19" gate="1" x="142.24" y="20.32"/>
+<instance part="R1" gate="G$1" x="149.86" y="25.4"/>
 </instances>
 <busses>
@@
 </segment>
 <segment>
-<pinref part="PARANI" gate="A" pin="1"/>
-<wire x1="241.3" y1="58.42" x2="226.06" y2="58.42" width="0.1524" layer="91"/>
-<label x="226.06" y="58.42" size="1.778" layer="95"/>
-</segment>
-<segment>
-<pinref part="PARANI" gate="A" pin="12"/>
-<wire x1="248.92" y1="45.72" x2="264.16" y2="45.72" width="0.1524" layer="91"/>
-<label x="256.54" y="45.72" size="1.778" layer="95"/>
-</segment>
-<segment>
-<pinref part="PARANI" gate="A" pin="9"/>
-<wire x1="241.3" y1="48.26" x2="226.06" y2="48.26" width="0.1524" layer="91"/>
-<label x="226.06" y="48.26" size="1.778" layer="95"/>
+<wire x1="213.36" y1="22.86" x2="220.98" y2="22.86" width="0.1524" layer="91"/>
+<wire x1="220.98" y1="22.86" x2="220.98" y2="20.32" width="0.1524" layer="91"/>
+<pinref part="GND13" gate="1" pin="GND"/>
+<pinref part="U$1" gate="G$1" pin="GND"/>
+</segment>
+<segment>
+<pinref part="R1" gate="G$1" pin="1"/>
+<pinref part="GND19" gate="1" pin="GND"/>
+<wire x1="144.78" y1="25.4" x2="142.24" y2="25.4" width="0.1524" layer="91"/>
+<wire x1="142.24" y1="25.4" x2="142.24" y2="22.86" width="0.1524" layer="91"/>
 </segment>
 </net>
@@
 </segment>
 <segment>
-<pinref part="PARANI" gate="A" pin="11"/>
-<wire x1="241.3" y1="45.72" x2="226.06" y2="45.72" width="0.1524" layer="91"/>
-<label x="226.06" y="45.72" size="1.778" layer="95"/>
+<wire x1="213.36" y1="25.4" x2="220.98" y2="25.4" width="0.1524" layer="91"/>
+<wire x1="220.98" y1="25.4" x2="220.98" y2="27.94" width="0.1524" layer="91"/>
+<pinref part="P+1" gate="G$1" pin="+3V3"/>
+<pinref part="U$1" gate="G$1" pin="VDD"/>
 </segment>
 </net>
@@
 <net name="RXD" class="0">
 <segment>
-<pinref part="PARANI" gate="A" pin="3"/>
-<wire x1="241.3" y1="55.88" x2="226.06" y2="55.88" width="0.1524" layer="91"/>
-<label x="226.06" y="55.88" size="1.778" layer="95"/>
-</segment>
-<segment>
 <pinref part="U1" gate="G$1" pin="(RXD1/AIN1/INT2)PD2"/>
 <wire x1="53.34" y1="73.66" x2="71.12" y2="73.66" width="0.1524" layer="91"/>
 <label x="63.5" y="73.66" size="1.778" layer="95"/>
 </segment>
+<segment>
+<pinref part="U$1" gate="G$1" pin="UART_TX"/>
+<wire x1="177.8" y1="-15.24" x2="170.18" y2="-15.24" width="0.1524" layer="91"/>
+<label x="170.18" y="-15.24" size="1.778" layer="95"/>
+</segment>
 </net>
 <net name="PB0" class="0">
@@
 <wire x1="53.34" y1="78.74" x2="71.12" y2="78.74" width="0.1524" layer="91"/>
 <label x="63.5" y="78.74" size="1.778" layer="95"/>
+</segment>
+<segment>
+<pinref part="STAND-BY" gate="G$1" pin="2"/>
+<wire x1="147.32" y1="53.34" x2="134.62" y2="53.34" width="0.1524" layer="91"/>
+<wire x1="134.62" y1="53.34" x2="134.62" y2="45.72" width="0.1524" layer="91"/>
+<wire x1="134.62" y1="45.72" x2="142.24" y2="45.72" width="0.1524" layer="91"/>
+<pinref part="R5" gate="G$1" pin="1"/>
+<wire x1="134.62" y1="53.34" x2="129.54" y2="53.34" width="0.1524" layer="91"/>
+<label x="129.54" y="53.34" size="1.778" layer="95"/>
+<junction x="134.62" y="53.34"/>
+</segment>
+</net>
+<net name="ADC10" class="0">
+<segment>
+<pinref part="U1" gate="G$1" pin="(T0/OC4D/ADC10)PD7"/>
+<wire x1="53.34" y1="86.36" x2="71.12" y2="86.36" width="0.1524" layer="91"/>
+<label x="63.5" y="86.36" size="1.778" layer="95"/>
 </segment>
 <segment>
@@
 </segment>
 </net>
-<net name="ADC10" class="0">
-<segment>
-<pinref part="STAND-BY" gate="G$1" pin="2"/>
-<wire x1="147.32" y1="53.34" x2="134.62" y2="53.34" width="0.1524" layer="91"/>
-<wire x1="134.62" y1="53.34" x2="134.62" y2="45.72" width="0.1524" layer="91"/>
-<wire x1="134.62" y1="45.72" x2="142.24" y2="45.72" width="0.1524" layer="91"/>
-<pinref part="R5" gate="G$1" pin="1"/>
-<wire x1="134.62" y1="53.34" x2="129.54" y2="53.34" width="0.1524" layer="91"/>
-<label x="129.54" y="53.34" size="1.778" layer="95"/>
-<junction x="134.62" y="53.34"/>
-</segment>
-<segment>
-<pinref part="U1" gate="G$1" pin="(T0/OC4D/ADC10)PD7"/>
-<wire x1="53.34" y1="86.36" x2="71.12" y2="86.36" width="0.1524" layer="91"/>
-<label x="63.5" y="86.36" size="1.778" layer="95"/>
-</segment>
-</net>
 <net name="ADC9" class="0">
 <segment>
@@
 <net name="TXD" class="0">
 <segment>
-<pinref part="PARANI" gate="A" pin="5"/>
-<wire x1="241.3" y1="53.34" x2="226.06" y2="53.34" width="0.1524" layer="91"/>
-<label x="226.06" y="53.34" size="1.778" layer="95"/>
-</segment>
-<segment>
 <wire x1="53.34" y1="76.2" x2="71.12" y2="76.2" width="0.1524" layer="91"/>
 <label x="63.5" y="76.2" size="1.778" layer="95"/>
 <pinref part="U1" gate="G$1" pin="(TXD1/INT3)PD3"/>
+</segment>
+<segment>
+<pinref part="U$1" gate="G$1" pin="UART_RX"/>
+<wire x1="177.8" y1="-17.78" x2="170.18" y2="-17.78" width="0.1524" layer="91"/>
+<label x="170.18" y="-17.78" size="1.778" layer="95"/>
 </segment>
 </net>
@@
 </segment>
 </net>
+<net name="N$7" class="0">
+<segment>
+<pinref part="STATUSLED" gate="G$1" pin="A"/>
+<pinref part="U$1" gate="G$1" pin="GPIO2"/>
+<wire x1="167.64" y1="25.4" x2="177.8" y2="25.4" width="0.1524" layer="91"/>
+</segment>
+</net>
+<net name="N$8" class="0">
+<segment>
+<pinref part="R1" gate="G$1" pin="2"/>
+<pinref part="STATUSLED" gate="G$1" pin="C"/>
+<wire x1="154.94" y1="25.4" x2="160.02" y2="25.4" width="0.1524" layer="91"/>
+</segment>
+</net>

Commit message: GloveMouse v2.2 all-in-one commit
Parts:
- removed JP3: AVR-JTAG-10, avr-7:AVR-JTAG-10
- removed LED3, LED6: GREEN, led:LEDCHIP-LED0805
- removed R22, R24: 1k, resistor:R-EU_R0603
- added JP1: AVR-ISP-6, avr-5:AVR-ISP-6
- GYRO: device pinhead:PINHD-1X7 -> pinhead:PINHD-1X5
Connections:
- removed net N$4: LED3.A, R22.1
- removed net N$6: LED6.A, R24.1
- removed net PB0: LED6.C, U1.(SS/PCINT0)PB0
- removed net PB1: LED5.C, U1.(SCLK/PCINT1)PB1
- removed net PB2: LED3.C, U1.(PDI/MOSI/PCINT2)PB2
- removed net PB3: LED4.C, U1.(PD0/MISO/PCINT3)PB3
- removed net PD0: GYRO.6, U1.(OC0B/SCL/INT0)PD0
- removed net PD1: GYRO.7, U1.(SDA/INT1)PD1
- removed net TCK: JP3.1, U1.(ADC4/TCK)PF4
- removed net TDI: JP3.9, U1.(ADC7/TDI)PF7
- removed net TDO: JP3.3, U1.(ADC6/TDO)PF6
- removed net TMS: JP3.5, U1.(ADC5/TMS)PF5
- new net ADC6: GYRO.3, U1.(ADC6/TDO)PF6
- new net ADC7: GYRO.4, U1.(ADC7/TDI)PF7
- new net MISO: JP1.1, U1.(PD0/MISO/PCINT3)PB3
- new net MOSI: JP1.4, U1.(PDI/MOSI/PCINT2)PB2
- new net PF0: LED4.A, U1.(ADC0)PF0
- new net PF1: LED5.A, U1.(ADC1)PF1
- new net SCK: JP1.3, U1.(SCLK/PCINT1)PB1
- net +3V3: now also JP1.2; no longer GYRO.2, JP3.4, JP3.7, R21.2, R22.2, R23.2, R24.2
- net GND: now also GYRO.2, JP1.6, R21.2, R23.2; no longer GYRO.3, JP3.10, JP3.2
- net N$1: now also LED5.C; no longer LED5.A
- net N$2: now also LED4.C; no longer LED4.A
- net RESET: now also JP1.5; no longer JP3.6
Other:
- note added: "Bluetooth"
- note added: "Vin + charger"
- note added: "microUSB"
- note added: "programator"
- note added: "uC"
- moved on the sheet: C11, C13, C15, C8, C9, IC3, J1, LED4, LED5, LEFT_CLICK, LIPO, ON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

Commit message: v3.0: initial commit for GloveMouse v3.0
Changed ATmega32U4 with ATmega128RFA1.
Added onboard gyroscope from v2.4.
Added battery level measuring system.
Added controlable power led and low-battery led.
Parts:
- removed C1, C2, C6: 100n, SmartPrj:C-EUC0603
- removed C3, C4: 22p, SmartPrj:C-EUC0603
- removed C5, C7: 1uF, SmartPrj:C-EUC0603
- removed GYRO: (no value), pinhead:PINHD-1X5
- removed L1: MH2029-300Y, wuerth-elektronik:WE-CBF_0805
- removed LED4: YELLOW, led:LEDCHIP-LED0805
- removed LED5, ON: GREEN, led:LEDCHIP-LED0805
- removed LEFT_CLICK, RIGHT_CLICK, STAND-BY: (no value), pinhead:PINHD-1X2
- removed Q2: (no value), crystal:CRYSTALCTS406
- removed RESET_SW, SENS_SELECT: (no value), switch-omron:10-XX
- removed SJ1: (no value), jumper:SJ
- removed STATUSLED: BLUE, led:LEDCHIP-LED0805
- removed U$1: RN42, Tudor's_spankin'_library:RN42
- removed U1: ATMEGA32U4-XUAU, SmartPrj:ATMEGA32U4-XUAU
- added C10: 100nF, resistor:C-EUC0603K
- added C12: 10uF, rcl:CPOL-EUSMCB
- added C14: 470nF, resistor:C-EUC0603K
- added C16: 10nF, resistor:C-EUC0603K
- added C17, C18: 0.1uF, resistor:C-EUC0603K
- added C19, C20, C23, C24: 22pF, resistor:C-EUC0603
- added C21, C22: 15pF, resistor:C-EUC0603
- added C25, C26, C27, C28: 100nF, resistor:C-EUC0603
- added LCLICK_BTN, RCLICK_BTN, STAND-BY_BTN: (no value), pinhead:PINHD-1X2/90
- added LOWBAT_LED: RED, led:LEDCHIP-LED0805
- added PWR_LED: GREEN, led:LEDCHIP-LED0805
- added Q1: ABM3B-16, 0andrei_custom:ABM3B-16
- added Q3: ABS25-32768, danode:ABS25-32768
- added R10: 10K, resistor:R-EU_R0603
- added R11, R12: 33K, resistor:R-EU_R0603
- added R14: 10k, resistor:R-EU_R0603
- added R15: 0, resistor:R-EU_R0603
- added RESET_BTN, SENS_BTN: (no value), switch-omron:10-XX
- added SENS0_LED, SENS1_LED: YELLOW, led:LEDCHIP-LED0805
- added U2: LPY403AL, Tudor's_spankin'_library:LPY403AL
- added U3: ANTENNA, 0andrei_custom:ANTENNA
- added U5: BALUN, 0andrei_custom:BALUN
- added U6: ATMEGA128RFA1, SparkFun:ATMEGA128RFA1
- C11, C15: value 1u -> 1uF; device SmartPrj:C-EUC0603 -> resistor:C-EUC0603K
- C13: value 10u -> 10uF; device rcl:C-EUC0603 -> resistor:C-EUC0603K
- C8: value 10u -> 10uF
- C9: value 100n -> 100nF; device SmartPrj:C-EUC0603 -> resistor:C-EUC0603K
- LIPO: device pinhead:PINHD-1X3 -> pinhead:PINHD-1X2/90
- R1: value 220 -> 100R
- R13: device SmartPrj:R-EU_R0603 -> resistor:R-EU_R0603
- R2, R21, R23: value 1k -> 100R
- R3, R4, R5, R6: value 100k -> 10k
- R7: value 10K -> 100k; device SmartPrj:R-EU_R0603 -> resistor:R-EU_R0603
- R8: value 22R -> 100k; device SmartPrj:R-EU_R0603 -> resistor:R-EU_R0603
- R9: value 22R -> 10k; device SmartPrj:R-EU_R0603 -> resistor:R-EU_R0603
Connections:
- removed net ADC10: LEFT_CLICK.2, R3.1, U1.(T0/OC4D/ADC10)PD7
- removed net ADC6: GYRO.3, U1.(ADC6/TDO)PF6
- removed net ADC7: GYRO.4, U1.(ADC7/TDI)PF7
- removed net ADC8: R5.1, STAND-BY.2, U1.(ICP1/ADC8)PD4
- removed net ADC9: R4.1, RIGHT_CLICK.2, U1.(T1/#OC4D/ADC9)PD6
- removed net AREF: C6.2, U1.AREF
- removed net AVCC: C5.1, L1.2, U1.AVCC, U1.AVCC1
- removed net D+: J1.D+, R9.1
- removed net D-: J1.D-, R8.1
- removed net HWB: R7.2, SJ1.1, U1.(#HWB)PE2
- removed net PB4: R6.1, SENS_SELECT.P, SENS_SELECT.P1, U1.(ADC11/PCINT4)PB4
- removed net PF0: LED4.A, U1.(ADC0)PF0
- removed net PF1: LED5.A, U1.(ADC1)PF1
- removed net RD+: R9.2, U1.D+
- removed net RD-: R8.2, U1.D-
- removed net RXD: U$1.UART_TX, U1.(RXD1/AIN1/INT2)PD2
- removed net TXD: U$1.UART_RX, U1.(TXD1/INT3)PD3
- removed net VUSB: C15.2, C8.+, C9.2, IC3.CE, IC3.PROG, IC3.VDD, J1.VBUS, U1.VBUS
- removed net XTAL1: C4.1, Q2.1, U1.XTAL1
- removed net XTAL2: C3.2, Q2.2, U1.XTAL2
- new net BAT: R7.2, R8.2, U6.PF7
- new net F1: C14.1, C16.1, U2.FILTVDD
- new net F2: C16.2, R10.1, U2.VCONT
- new net LCLICK: LCLICK_BTN.2, R3.2, U6.PF2
- new net LOWBAT: R1.1, U6.PG5
- new net N$10: C18.1, R11.2, U2.4XIN_X
- new net N$11: C21.1, Q3.$, U6.PG3
- new net N$12: C22.1, Q3.2, U6.PG4
- new net N$13: C24.2, U6.RFP
- new net N$14: C23.2, U6.RFN
- new net N$15: C23.1, U5.BAL1
- new net N$16: C24.1, U5.BAL2
- new net N$17: C25.1, U6.DVDD@21, U6.DVDD@22
- new net N$18: C26.1, U6.AVDD
- new net N$19: R9.2, U6.TST
- new net N$20: R15.1, U5.UNBAL
- new net N$21: R14.2, U6.CLKI
- new net N$22: R15.2, U3.P$1
- new net N$4: C14.2, R10.2
- new net N$6: R12.1, U2.OUT_Z
- new net N$9: C19.1, Q1.XTAL1, U6.XTAL1
- new net PWR: R2.1, U6.PB7
- new net RCLICK: R4.2, RCLICK_BTN.2, U6.PF3
- new net SENS: R6.1, SENS_BTN.P, SENS_BTN.P1
- new net SENS0: R21.1
- new net SENS1: R23.1
- new net STAND-BY: R5.2, STAND-BY_BTN.2, U6.PF4
- new net VBAT: C13.1, IC3.VBAT, LIPO.1, R7.1, U4.VIN
- new net VBUS: C15.1, C8.+, C9.1, IC3.CE, IC3.PROG, IC3.VDD, J1.VBUS
- new net XGYRO: U2.4XOUT_X, U6.PF5
- new net XOUT-1X2: C17.1, R12.2, U2.4XIN_Z
- new net ZGYRO: U2.4XOUT_Z, U6.PF6
- net +3V3: now also C10.1, C11.1, C12.+, C27.1, C28.1, R3.1, R4.1, R5.1, U2.VDD, U2.VDD_2, U6.AREF, U6.DEVDD@23, U6.DEVDD@34, U6.DEVDD@44, U6.DEVDD@54, U6.EVDD; no longer C1.1, C11.2, C2.1, C7.1, GYRO.1, L1.1, R2.1, R3.2, R4.2, R5.2, R7.1, U$1.VDD, U1.UCAP, U1.UVCC, U1.VCC, U1.VCC1
- net GND: now also C10.2, C11.2, C12.-, C13.2, C15.2, C17.2, C18.2, C19.2, C20.2, C21.2, C22.2, C25.2, C26.2, C27.2, C28.2, C9.2, LCLICK_BTN.1, LOWBAT_LED.C, PWR_LED.C, Q1.GND1, Q1.GND2, Q3.GND1, Q3.GND2, R14.1, R8.1, R9.1, RCLICK_BTN.1, RESET_BTN.S, RESET_BTN.S1, SENS0_LED.C, SENS1_LED.C, SENS_BTN.S, SENS_BTN.S1, STAND-BY_BTN.1, U2.GND, U2.HP, U2.SLEEP/PD, U2.ST, U5.GND, U6.AVSS@58, U6.AVSS@61, U6.AVSS_RFN, U6.AVSS_RFP, U6.DVSS@20, U6.DVSS@24, U6.DVSS@35, U6.DVSS@45, U6.DVSS@55; no longer C1.2, C11.1, C13.1, C15.1, C2.2, C3.1, C4.2, C5.2, C6.1, C7.2, C9.1, GYRO.2, LEFT_CLICK.1, ON.C, R1.1, R21.2, R23.2, RESET_SW.S, RESET_SW.S1, RIGHT_CLICK.1, SENS_SELECT.S, SENS_SELECT.S1, SJ1.2, STAND-BY.1, U$1.GND, U1.GND, U1.GND1, U1.GND2, U1.GND3, U1.PAD, U1.UGND
- net MISO: now also U6.PB3/PDO; no longer U1.(PD0/MISO/PCINT3)PB3
- net MOSI: now also U6.PB2/PDI; no longer U1.(PDI/MOSI/PCINT2)PB2
- net N$1: now also R23.2, SENS1_LED.A; no longer LED5.C, R23.1
- net N$2: now also LOWBAT_LED.A, R1.2; no longer LED4.C, R21.1
- net N$3: now also PWR_LED.A; no longer ON.A
- net N$5: now also R21.2, SENS0_LED.A; no longer C13.2, IC3.VBAT, LIPO.1, U4.VIN
- net N$7: now also R11.1, U2.OUT_X; no longer STATUSLED.A, U$1.GPIO2
- net N$8: now also C20.1, Q1.XTAL2, U6.XTAL2; no longer R1.2, STATUSLED.C
- net RESET: now also RESET_BTN.P, RESET_BTN.P1, U6.RSTN; no longer RESET_SW.P, RESET_SW.P1, U1.RESET
- net SCK: now also U6.PB1/SCK; no longer U1.(SCLK/PCINT1)PB1
Other:
- note added: "Battery"
- note added: "Battery meter"
- note added: "Buttons"
- note added: "Charger"
- note added: "Gyroscope"
- note added: "Indicator LEDs"
- note added: "Input"
- note added: "Sensitivity"
- note added: "Supply"
- note added: "Voltage regulator"
- note removed: "Bluetooth"
- note removed: "Gyro connector"
- note removed: "Sensitivity LEDs"
- note removed: "Sensitivity select button"
- note removed: "To Own Battery"
- note removed: "Touch buttons"
- note removed: "Vin + charger"
- note removed: "programator"
- moved on the sheet: C11, C13, C15, C8, C9, IC3, J1, JP1, R1, R13, R2, R21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

Commit message: v3.0 release candidate 1
Changed secondary crystal.
Finished routing.
Parts:
- removed Q3: ABS25-32768, danode:ABS25-32768
- removed R15: 0, resistor:R-EU_R0603
- added Q2: 32.768kHz, crystal:FC-12M
Connections:
- removed net N$20: R15.1, U5.UNBAL
- net GND: now also LCLICK_BTN.2, RCLICK_BTN.2, STAND-BY_BTN.2; no longer LCLICK_BTN.1, Q3.GND1, Q3.GND2, RCLICK_BTN.1, STAND-BY_BTN.1
- net LCLICK: now also LCLICK_BTN.1, U6.PF3; no longer LCLICK_BTN.2, U6.PF2
- net N$11: now also Q2.2; no longer Q3.$
- net N$12: now also Q2.1; no longer Q3.2
- net N$22: now also U5.UNBAL; no longer R15.2
- net RCLICK: now also RCLICK_BTN.1, U6.PF6; no longer RCLICK_BTN.2, U6.PF3
- net SENS: now also U6.PE3
- net SENS0: now also U6.PE5
- net SENS1: now also U6.PE4
- net STAND-BY: now also STAND-BY_BTN.1, U6.PF5; no longer STAND-BY_BTN.2, U6.PF4
- net XGYRO: now also U6.PF2; no longer U6.PF5
- net ZGYRO: now also U6.PF4; no longer U6.PF6
Other:
- note added: "ISP"
- note added: "Reset button"
- moved on the sheet: C19, C20, C21, C22, C23, C24, C25, C26, C27, C28, JP1, LCLICK_BTN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
